File: schematics/Pro Trinket Keyboard V3.1.brd (EAGLE design)
At the start: 80 x 80 mm, 45 parts, among them SW10 ROTARTY_ENCODER, SW11 ROTARTY_ENCODER, SW12 ROTARTY_ENCODER, SW9 ROTARTY_ENCODER

Commit message: updated schematic and layout
Parts:
- ZENER1, ZENER2: device SparkFun-DiscreteSemi:SOD-323 -> diode:SOD80C
- moved C1 15.1 mm to (40.2, 76.5), turned to 180 degrees
- moved R5 2.29 mm to (62.9, 68.9), turned to 0 degrees
- moved R6 2.03 mm to (65.7, 67.6), turned to 0 degrees
- moved ZENER2 1.00 mm to (69.5, 72.7)
- moved ZENER1 0.71 mm to (67.6, 70.5)
- moved C2 0.40 mm to (38.6, 61.2)
- moved R4 0.32 mm to (65.4, 73.0)
- moved JP1 0.19 mm to (67.3, 77.3)
Connections:
- net A6: now also U$2.A6
- net AREF: now also U$2.AREF
Routing:
- net A6: track 2.19 -> 9.38 mm, vias 0 -> 1
- net D7/D-: track 24.0 -> 20.4 mm
- net N$12: track 5.12 -> 8.29 mm
- net AREF: track 4.17 -> 6.84 mm
- net D2/D+: track 38.5 -> 35.9 mm
- net N$11: track 5.32 -> 7.68 mm
- net N$2: track 36.0 -> 36.5 mm
- net L31: track 36.0 -> 36.5 mm
- net GND: track 16.8 -> 16.7 mm, vias 26 -> 29
Other:
- board text added: "hackaday.io/project/3502 v3.1 03/2015"
