File: schematics/Pro Trinket Keyboard V3.1.sch (EAGLE design)
At the start: 44 parts, among them SW10 ROTARTY_ENCODER, SW11 ROTARTY_ENCODER, SW12 ROTARTY_ENCODER, SW9 ROTARTY_ENCODER

Commit message: updated schematic and layout
Parts:
- ZENER1, ZENER2: device SparkFun-DiscreteSemi:DIODE-ZENER-BZT52 -> diode:ZENER-DIODESOD80C
Connections:
- net A6: now also U$2.A6
- net AREF: now also U$2.AREF
Other:
- moved on the sheet: C9, L11, L12, L21, L22, L31, L32, MODE, R1, R2, R3
