File: schematics/Pro Trinket Keyboard V3.4.brd (EAGLE design)
At the start: 80 x 80 mm, 79 parts

Commit message: updated board file
Routing:
- net D12: track 86.9 -> 88.8 mm
- net A0/D14: track 72.1 -> 70.5 mm
- net GND: vias 56 -> 71
